File: Design/Smart_Plant.sch (EAGLE design)
At the start: 22 parts, among them IC1 555

Commit message: Added design files for 'Kit' branch
Parts:
- removed C1: 10nF, rcl:C-US050-025X075
- removed C2: 470pF, rcl:C-US050-025X075
- removed C3: 1uF, rcl:CPOL-USE2.5-5
- removed D1: 1N4004, diode:1N4004
- removed H1, H2: MOUNT-PAD-ROUND3.0, holes:MOUNT-PAD-ROUND3.0
- removed IC1: 555, SparkFun-IC-Special-Function:555KIT
- removed JMP1: 0R-JUMPB, jump-0r-smd:0R-JUMPB
- removed LDR: VT20N1, photo-elements:VT20N1
- removed NTC: R1206, ptc-ntc:NTC640
- removed R1, R2, R6, R8: 10k, rcl:R-US_0207/10
- removed R3: 1k, rcl:R-US_0207/10
- removed R4: 330, rcl:R-US_0207/10
- removed R5: 1k6, rcl:R-US_0207/10
- removed R7: 1M, rcl:R-US_0207/10
- removed SJ1: (no value), jumper:SJ
- removed T1: (no value), transistor:-NPN-TO92-ECB
- added J1: 455-1750-1-ND, SparkFun-Connectors:CONN_03
- added J2, J3: (no value), SparkFun-Connectors:CONN_04PTH
Connections:
- removed net EC_1: H1.MOUNT, JP1.8
- removed net EC_2: H2.MOUNT, JP1.9, R8.2
- removed net EXC: JMP1-0R.1, JP1.12, R3.2
- removed net LIGHT: JP2.10, LDR.2, R1.2
- removed net MOIST: C3.+, D1.C, JP2.9, R7.1, SJ1.1
- removed net N$1: R3.1, T1.B
- removed net N$10: JMP1-0R.3, T1.E
- removed net N$3: C2.1, IC1.TRE, IC1.TRI, R5.2
- removed net N$4: IC1.DIS, R4.2, R5.1
- removed net N$6: IC1.OUT, R6.1
- removed net N$9: C1.2, IC1.CON
- removed net SIG: D1.A, R6.2, SJ1.2
- removed net TEMP: JP2.11, NTC.1, R2.2
- removed net VSENS: IC1./RES, IC1.VCC+, JMP1-0R.2, LDR.1, NTC.2, R4.1
- new net A0: J1.3, JP1.1
- new net SCL: J2.2, J3.2, JP2.6
- new net SDA: J2.1, J3.1, JP2.3
- net 3V3: now also J1.2, J2.4, J3.4; no longer T1.C
- net GND: now also J1.1, J2.3, J3.3; no longer C1.1, C2.2, C3.-, IC1.GND, R1.1, R2.1, R7.2, R8.1
Other:
- note removed: "B.1.0 - SMD 1206 B.1.1 - THT B.2.0 - NO 555 THT"
- note removed: "Version:"

Commit message: Added design files to 'Custom' branch
Parts:
- removed J1: 455-1750-1-ND, SparkFun-Connectors:CONN_03
- removed J2, J3: (no value), SparkFun-Connectors:CONN_04PTH
- removed JP2: (no value), SparkFun-Connectors:CONN_13
- added C1, C2, C3, C34, C37, C38, C41, C48, C49, C51, C53: 0.1uF, SparkFun-Capacitors:0.1UF-0603-25V-(+80/-20%)
- added C13, C14, C17, C18, C19, C25, C27, C28, C9: 1uF, microbuilder:CAP_CERAMIC0805-NOOUTLINE
- added C26: 4.7uF/25V, microbuilder:CAP_CERAMIC0805-NOOUTLINE
- added C29, C30: 10pF, SparkFun-Capacitors:10PF-0603-50V-5%
- added C31, C32: 270pF, esp32-thing-temp:270PF-50V-5%(0603)
- added C33: 10nF, SparkFun-Capacitors:10NF-0603-50V-10%
- added C35: 2.4pF, esp32-thing-temp:2.4PF-0603-50V-5%
- added C36: 5.6pF, esp32-thing-temp:5.6PF-50V-5%(0603)
- added C39, C40: 47pF, SparkFun-Capacitors:47PF-0603-50V-5%
- added C42: 4.7uF, SparkFun-Capacitors:4.7UF-6.3V-10%(0603)0603
- added C43: 1.0uF, SparkFun-Capacitors:1.0UF-0805-25V-(+80/-20%)
- added C44: 2.2uF, SparkFun-Capacitors:2.2UF-0603-10V-20%
- added C45, C46: 4.7uF, SparkFun-Capacitors:4.7UF0603
- added C47: 100pF, SparkFun-Capacitors:100PF-0603-50V-5%
- added C50: 10uF, SparkFun-Capacitors:10UF-0603-6.3V-20%
- added C52: 1.0uF, SparkFun-Capacitors:1.0UF-0603-16V-10%
- added C56: 3.0nF, esp32-thing-temp:3.0NF-0603-50V-5%
- added C8: 10uF/10V+, microbuilder:CAP_CERAMIC0805-NOOUTLINE
- added D10, D4, D9: MBR0530, microbuilder:DIODE-SCHOTTKYSOD-123
- added D5: BAT20J, SparkFun-DiscreteSemi:DIODE-SCHOTTKY-BAT20J
- added D6: Yellow, SparkFun-LED:LED-YELLOW0603
- added D7: Green, SparkFun-LED:LED-RED0603
- added E2: ANTENNA, esp32-thing-temp:ANTENNATRACE-TUNED
- added EINK1: EINK_24PIN_290IN, microbuilder:EINK_24PIN_290IN
- added F2: 500mA, SparkFun-PowerIC:PTCSMD
- added IC1: NE555D, linear:NE555D
- added JP3: LiPo, SparkFun-Connectors:M02JST-PTH-2
- added L2: 2.7nH, SparkFun-Passives:INDUCTOR0603
- added L3: 10uH, microbuilder:INDUCTORNR401
- added Q1: IRLML0100, Parts:IRLML2060TRPBF
- added Q3: 2.5A/30V, SparkFun-DiscreteSemi:MOSFET-PCHANNELDMG2307L
- added Q4: MBT3904DW1T1, esp32-thing-temp:MBT3904DW1T1
- added R1, R12, R15, R2, R3: 27, SparkFun-Resistors:27OHM1/10W1%(0603)0603-RES
- added R10, R26: 10k, SparkFun-Resistors:10KOHM-1/10W-1%(0603)0603
- added R11: 20k, SparkFun-Resistors:20KOHM-0603-1/10W-1%
- added R13: 0.47ohm, microbuilder:RESISTOR0805_10MGAP
- added R16, R22, R23: 10k, SparkFun-Resistors:10KOHM-0603-1/10W-1%
- added R19, R24: 1K, SparkFun-Resistors:1KOHM-1/10W-1%(0603)
- added R20: 2.0k, SparkFun-Resistors:2.0KOHM1/10W5%(0603)
- added R21: DNP, SparkFun-Passives:RESISTORPTH-1/6W
- added R27: DNP, microbuilder:RESISTOR0805_10MGAP
- added S3: RESET, SparkFun-Electromechanical:SWITCH-MOMENTARY-2SMD-4.6X2.8MM
- added S4: BTN-0, SparkFun-Electromechanical:SWITCH-MOMENTARY-2SMD-4.6X2.8MM
- added SJ4: JUMPER-PAD-3-2OF3_NC_BY_TRACE_SMALL, SparkFun-Passives:JUMPER-PAD-3-2OF3_NC_BY_TRACE_SMALL
- added SJ5: JUMPER-PAD-2-NC_BY_TRACE, SparkFun-Passives:JUMPER-PAD-2-NC_BY_TRACE
- added U10: ESP3212, esp32-thing-temp:ESP3212
- added U6: W25Q32FVSS, SparkFun-DigitalIC:W25Q32FVSS
- added U7: FT231XS, SparkFun-DigitalIC:FT231XS
- added U8: MCP73831, SparkFun-PowerIC:MCP73831
- added U9: AP2112K-3.3V, SparkFun-PowerIC:V_REG_LDOSMD
- added X2: MICROSD, microbuilder:MICROSD
- added Y3: 26MHz, things:CRYSTAL-GROUNDED3.2X2.5
- JP1: device SparkFun-Connectors:CONN_13 -> SparkFun-Connectors:USB_MICROB_PLUGCONN-11752
Connections:
- removed net A0: J1.3, JP1.1
- removed net SCL: J2.2, J3.2, JP2.6
- removed net SDA: J2.1, J3.1, JP2.3
- new net 0: Q4Q2.C, R26.1, S4.2, U10.(ADC2:1/TOUCH1/RTC11/CLK_OUT1)GPIO0
- new net 12: U10.(GPIO12/ADC2:5/TOUCH5/RTC15/SPIQ)MTDI
- new net 19: U10.(VSPIQ/HS2_DATA2)GPIO19
- new net 21: U10.(VSPIHD/HS2_CMD)GPIO21
- new net 22: U10.(VSPIWP/HS2_CLK)GPIO22
- new net 25: U10.(DAC1/ADC2:8/RTC6)GPIO25
- new net 26: U10.(DAC2/ADC2:9/RTC7)GPIO26
- new net 27: U10.(ADC2:7/TOUCH7/RTC17)GPIO27
- new net 3.3V_F: C41.1, U7.!RESET, U7.3V3OUT, U7.VCCIO
- new net 32: U10.32K_XP(GPIO32/ADC1:4/TOUCH9/RTC9)
- new net 33: U10.32K_XN(GPIO33/ADC1:5/TOUCH8/RTC8)
- new net 34: U10.VDET_1(GPI34/ADC1:6)
- new net 35: U10.VDET_2(GPI35/ADC1:7)
- new net 36: C31.2, U10.SENSOR_VP(GPI36/ADC1:0/RTC0)
- new net 37: C31.1, U10.SENSOR_CAPP(GPI37/ADC1:1/RTC1)
- new net 38: C32.1, U10.SENSOR_CAPN(GPI38/ADC1:2/RTC2)
- new net 39: C32.2, U10.SENSOR_VN(GPI39/ADC1:3/RTC3)
- new net BUSY: EINK1.BUSY, U10.(ADC2:0/TOUCH0/RTC10/SPIHD)GPIO4
- new net CAP_10N1: C33.2, C56.1, R11.2, U10.CAP1
- new net CHIP_PU: Q4Q1.C, R10.1, S3.2, U10.CHIP_PU
- new net D+: C39.1, JP1.D+, R15.1
- new net D-: C40.1, JP1.D-, R12.1
- new net DC: EINK1.D/C#, U10.(HS1_DATA5)GPIO17
- new net DISPCS: EINK1.CS#, U10.(VSPICS0/HS1_DATA6)GPIO5
- new net DTR: Q4Q2.E, R22.1, U7.!DTR
- new net FLASH_SCK: U10.(GPIO6/SPICLK/HS1_CLK/U1CTS)SD_CLK, U6.SCK
- new net FLASH_SCS: U10.(GPIO11/SPICSO/HS1_CMD/U1RTS)SD_CMD, U6.!CS!
- new net FLASH_SDI: U10.(GPIO8/SPID/HS1_DATA1)SD_DATA1, U6.SI(D0)
- new net FLASH_SDO: U10.(GPIO7/SPI1/HS1_DATA0)SD_DATA0, U6.SO(D1)
- new net FLASH_SHD: U10.(GPIO9/SPIHD/HS1_DATA2/U1RX)SD_DATA2, U6.!HOLD!(D3)
- new net FLASH_SWP: U10.(GPIO10/SPIWP/HS1_DATA3/U1TX)SD_DATA3, U6.!WP!(D2)
- new net FLASH_VDD: C52.1, SJ4.1, U10.VDD3P3_SDIO
- new net GDR: EINK1.GDR, Q1.G
- new net LNA_IN1: C36.1, L2.1, U10.LNA_IN
- new net MISO_SD: U10.(ADC2:2/TOUCH2/RTC12/SPIWP)GPIO2, X2.DATA_OUT
- new net MOSI: EINK1.SDIO, U10.GPIO23
- new net MOSI_SD: U10.(GPIO15/ADC2:3/TOUCH3/RTC13/SPICSO/U0RTS)MTDO, X2.DATA_IN
- new net N$11: C9.2, EINK1.VSH2
- new net N$12: C13.2, EINK1.VDD
- new net N$13: C14.2, EINK1.VSH1
- new net N$14: C17.2, EINK1.VSL
- new net N$15: C18.2, EINK1.VCOM
- new net N$16: C26.2, D4.A, D9.C
- new net N$17: C26.1, D10.A, L3.1, Q1.D
- new net N$18: R15.2, U7.USBDP
- new net N$19: D6.A, R19.2
- new net N$20: D6.C, U8.STAT
- new net N$21: R21.2, SJ5.2, U8.PROG
- new net N$22: R20.2, SJ5.1
- new net N$23: Q4Q1.B, R22.2
- new net N$24: Q4Q2.B, R23.2
- new net N$25: C29.2, U10.XTAL_P, Y3.1
- new net N$26: C30.2, U10.XTAL_N, Y3.2
- new net N$27: D7.A, R24.2
- new net N$30: C56.2, R11.1, U10.CAP2
- new net N$31: C27.2, EINK1.VGL/NC
- new net N$32: C28.2, EINK1.VPP
- new net N$5: C34.1, SJ4.2, U6.VCC
- new net N$6: R12.2, U7.USBDM
- new net RESE: EINK1.RESE, Q1.S, R13.1, R27.1
- new net RESET: EINK1.RES#, U10.(HS1_DATA4)GPIO16
- new net RTS: Q4Q1.E, R23.1, U7.!RTS
- new net SCLK: EINK1.SCK, U10.(VSPICLK/HS1_DATA7)GPIO18
- new net SCLK_SD: U10.(GPIO14/ADC2:6/TOUCH6/RTC16/SPICLK)MTMS, X2.SCLK
- new net SDCS_SD: U10.(GPIO13/ADC2:4/TOUCH4/RTC14/SPID/U0CTS)MTCK, X2.CS
- new net SHIELD: JP1.SHIELD
- new net TRACE_ANT1: C35.1, C36.2, E2.SIGNAL
- new net TSCL: EINK1.TSCL
- new net TSDA: EINK1.TSDA
- new net U0RXD: U10.(GPIO3/CLK_OUT2/HS2_DATA0)U0RXD, U7.TXD
- new net U0TXD: U10.(GPIO1/CLK_OUT3/HS2_DATA1)U0TXD, U7.RXD
- new net VGH: C19.1, D10.C, EINK1.VGH
- new net VGL: C25.1, D9.A, EINK1.VGL
- new net VIN: C43.1, D5.C, Q3.S, U9.EN, U9.IN
- new net VUSB-RAW: C37.1, F2.1, JP1.VCC
- new net V_BATT: C45.1, JP3.2, Q3.D, U8.VBAT
- new net V_USB: C38.1, C42.1, C46.1, D5.A, F2.2, Q3.G, R16.2, R19.1, U7.VCC, U8.VIN
- net 3V3: now also C44.1, C47.1, C48.1, C49.1, C50.1, C51.1, C53.1, C8.2, EINK1.VCI, EINK1.VDDIO, L3.2, R10.2, R24.1, R26.2, SJ4.3, U10.VDD3P3_CPU, U10.VDD3P3_RTC, U10.VDDA, U10.VDDA3P3, U9.OUT, X2.SD_VDD; no longer J1.2, J2.4, J3.4, JP1.5
- net GND: now also C13.1, C14.1, C17.1, C18.1, C19.2, C25.2, C27.1, C28.1, C29.1, C30.1, C33.1, C34.2, C35.2, C37.2, C38.2, C39.2, C40.2, C41.2, C42.2, C43.2, C44.2, C45.2, C46.2, C47.2, C48.2, C49.2, C50.2, C51.2, C52.2, C53.2, C8.1, C9.1, D4.C, D7.C, E2.GND, EINK1.BSI, EINK1.VSS, JP1.GND, JP3.1, L2.2, R13.2, R16.1, R20.1, R21.1, R27.2, S3.1, S4.1, U10.GND, U6.GND, U7.GND@16, U7.GND@6, U8.VSS, U9.GND, X2.GND@1, X2.GND@2, X2.GND@3, Y3.GND; no longer J1.1, J2.3, J3.3, JP1.13
Other:
- note removed: "J.G.Aguado"
