File: Design/Smart_Plant.kicad_sch (KiCad schematic)
At the start: 38 parts, among them IC1 TP4056, IC4 RT9080-33GJ5, IC5 ESP32-S2-MINI-1-N4R2, J1 BAT_CONN-JST-2MM-SMT, J5 CONN_04PTH, Q1 IRLML0100

Commit message: V2R2 (XL): larger Smart Plant board variant
KiCad schematic/PCB/project updated for the XL version, GND fix,
fabrication toolkit options and production outputs (BOM, positions,
netlist, gerber zip), plus refreshed silkscreen documentation.

Co-Authored-By: Claude Opus 5.5 <noreply@anthropic.com>
Parts:
- renumbered FPC0 to FPC
Changed lines of the file:
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@@
 		(in_pos_files yes)
 		(dnp no)
-		(property "Reference" "FPC0"
+		(property "Reference" "FPC"
 			(at 254 39.37 0)
 			(show_name no)
@@
 			(project "Smart_Plant"
 				(path "/f81eaaab-182d-40b6-aa67-993c089e3c14"
-					(reference "FPC0")
+					(reference "FPC")
 					(unit 1)
 				)
